Commit message: some joint were manually fixed on the urdf file - changed taht so dimension is the same between model and trajectory

File: robot_models/biped_assets/biped_assets/models/h12/h12_12dof.urdf (robot description, URDF)
Before this commit: robot h1_5, 56 links, 55 joints
Links:
- added link world
Joints:
- added joint floating_base_joint: type floating, parent world, child pelvis
- joint left_elbow_joint: type fixed -> revolute
- joint left_shoulder_pitch_joint: type fixed -> revolute
- joint left_shoulder_roll_joint: type fixed -> revolute
- joint left_shoulder_yaw_joint: type fixed -> revolute
- joint left_wrist_pitch_joint: type fixed -> revolute
- joint left_wrist_roll_joint: type fixed -> revolute
- joint left_wrist_yaw_joint: type fixed -> revolute
- joint right_elbow_joint: type fixed -> revolute
- joint right_shoulder_pitch_joint: type fixed -> revolute
- joint right_shoulder_roll_joint: type fixed -> revolute
- joint right_shoulder_yaw_joint: type fixed -> revolute
- joint right_wrist_pitch_joint: type fixed -> revolute
- joint right_wrist_roll_joint: type fixed -> revolute
- joint right_wrist_yaw_joint: type fixed -> revolute
- joint torso_joint: type fixed -> revolute
