Commit message: model(h1_v2): simplified strucutre and use of robot from unity repos without arm

File: robot_models/h1_2_description/h1_2.urdf (robot description, URDF)
Before this commit: robot h1_5, 56 links, 55 joints
Links:
- added link camera_link
- added link lidar_link
- link L_hand_base_link: geometry collision mesh filename=meshes/L_hand_base_link.STL; visual mesh filename=meshes/L_hand_base_link.STL
- link L_index_intermediate: geometry collision mesh filename=meshes/link16_L.STL; visual mesh filename=meshes/link16_L.STL
- link L_index_proximal: geometry collision mesh filename=meshes/link15_L.STL; visual mesh filename=meshes/link15_L.STL
- link L_middle_intermediate: geometry collision mesh filename=meshes/link18_L.STL; visual mesh filename=meshes/link18_L.STL
- link L_middle_proximal: geometry collision mesh filename=meshes/link17_L.STL; visual mesh filename=meshes/link17_L.STL
- link L_pinky_intermediate: geometry collision mesh filename=meshes/link22_L.STL; visual mesh filename=meshes/link22_L.STL
- link L_pinky_proximal: geometry collision mesh filename=meshes/link21_L.STL; visual mesh filename=meshes/link21_L.STL
- link L_ring_intermediate: geometry collision mesh filename=meshes/link20_L.STL; visual mesh filename=meshes/link20_L.STL
- link L_ring_proximal: geometry collision mesh filename=meshes/link19_L.STL; visual mesh filename=meshes/link19_L.STL
- link L_thumb_distal: geometry collision mesh filename=meshes/link14_L.STL; visual mesh filename=meshes/link14_L.STL
- link L_thumb_intermediate: geometry collision mesh filename=meshes/link13_L.STL; visual mesh filename=meshes/link13_L.STL
- link L_thumb_proximal: geometry collision mesh filename=meshes/link12_L.STL; visual mesh filename=meshes/link12_L.STL
- link L_thumb_proximal_base: geometry collision mesh filename=meshes/link11_L.STL; visual mesh filename=meshes/link11_L.STL
- link R_hand_base_link: geometry collision mesh filename=meshes/R_hand_base_link.STL; visual mesh filename=meshes/R_hand_base_link.STL
- link R_index_intermediate: geometry collision mesh filename=meshes/link16_R.STL; visual mesh filename=meshes/link16_R.STL
- link R_index_proximal: geometry collision mesh filename=meshes/link15_R.STL; visual mesh filename=meshes/link15_R.STL
- link R_middle_intermediate: geometry collision mesh filename=meshes/link18_R.STL; visual mesh filename=meshes/link18_R.STL
- link R_middle_proximal: geometry collision mesh filename=meshes/link17_R.STL; visual mesh filename=meshes/link17_R.STL
- link R_pinky_intermediate: geometry collision mesh filename=meshes/link22_R.STL; visual mesh filename=meshes/link22_R.STL
- link R_pinky_proximal: geometry collision mesh filename=meshes/link21_R.STL; visual mesh filename=meshes/link21_R.STL
- link R_ring_intermediate: geometry collision mesh filename=meshes/link20_R.STL; visual mesh filename=meshes/link20_R.STL
- link R_ring_proximal: geometry collision mesh filename=meshes/link19_R.STL; visual mesh filename=meshes/link19_R.STL
- link R_thumb_distal: geometry collision mesh filename=meshes/link14_R.STL; visual mesh filename=meshes/link14_R.STL
- link R_thumb_intermediate: geometry collision mesh filename=meshes/link13_R.STL; visual mesh filename=meshes/link13_R.STL
- link R_thumb_proximal: geometry collision mesh filename=meshes/link12_R.STL; visual mesh filename=meshes/link12_R.STL
- link R_thumb_proximal_base: geometry collision mesh filename=meshes/link11_R.STL; visual mesh filename=meshes/link11_R.STL
- link left_ankle_pitch_link: geometry collision mesh filename=meshes/left_ankle_pitch_link.STL; visual mesh filename=meshes/left_ankle_pitch_link.STL
- link left_ankle_roll_link: geometry collision mesh filename=meshes/left_ankle_roll_link.STL; visual mesh filename=meshes/left_ankle_roll_link.STL
- link left_elbow_link: geometry collision mesh filename=meshes/left_elbow_link.STL; visual mesh filename=meshes/left_elbow_link.STL
- link left_hip_pitch_link: geometry collision cylinder length=0.2 radius=0.02; visual mesh filename=meshes/left_hip_pitch_link.STL
- link left_hip_roll_link: geometry collision cylinder length=0.01 radius=0.02; visual mesh filename=meshes/left_hip_roll_link.STL
- link left_hip_yaw_link: geometry collision cylinder length=0.02 radius=0.01; visual mesh filename=meshes/left_hip_yaw_link.STL
- link left_knee_link: geometry collision cylinder length=0.2 radius=0.02; visual mesh filename=meshes/left_knee_link.STL
- link left_shoulder_pitch_link: geometry collision mesh filename=meshes/left_shoulder_pitch_link.STL; visual mesh filename=meshes/left_shoulder_pitch_link.STL
- link left_shoulder_roll_link: geometry collision mesh filename=meshes/left_shoulder_roll_link.STL; visual mesh filename=meshes/left_shoulder_roll_link.STL
- link left_shoulder_yaw_link: geometry collision mesh filename=meshes/left_shoulder_yaw_link.STL; visual mesh filename=meshes/left_shoulder_yaw_link.STL
- link left_wrist_pitch_link: geometry collision mesh filename=meshes/left_wrist_pitch_link.STL; visual mesh filename=meshes/left_wrist_pitch_link.STL
- link left_wrist_roll_link: geometry collision mesh filename=meshes/left_wrist_roll_link.STL; visual mesh filename=meshes/left_wrist_roll_link.STL
- link left_wrist_yaw_link: geometry visual mesh filename=meshes/wrist_yaw_link.STL
- link logo_link: geometry visual mesh filename=meshes/logo_link.STL
- link pelvis: geometry collision sphere radius=0.05; visual mesh filename=meshes/pelvis.STL
- link right_ankle_pitch_link: geometry collision mesh filename=meshes/right_ankle_pitch_link.STL; visual mesh filename=meshes/right_ankle_pitch_link.STL
- link right_ankle_roll_link: geometry collision mesh filename=meshes/right_ankle_roll_link.STL; visual mesh filename=meshes/right_ankle_roll_link.STL
- link right_elbow_link: geometry collision mesh filename=meshes/right_elbow_link.STL; visual mesh filename=meshes/right_elbow_link.STL
- link right_hip_pitch_link: geometry collision cylinder length=0.2 radius=0.02; visual mesh filename=meshes/right_hip_pitch_link.STL
- link right_hip_roll_link: geometry collision cylinder length=0.01 radius=0.02; visual mesh filename=meshes/right_hip_roll_link.STL
- link right_hip_yaw_link: geometry collision cylinder length=0.02 radius=0.01; visual mesh filename=meshes/right_hip_yaw_link.STL
- link right_knee_link: geometry collision cylinder length=0.2 radius=0.02; visual mesh filename=meshes/right_knee_link.STL
- link right_shoulder_pitch_link: geometry collision mesh filename=meshes/right_shoulder_pitch_link.STL; visual mesh filename=meshes/right_shoulder_pitch_link.STL
- link right_shoulder_roll_link: geometry collision mesh filename=meshes/right_shoulder_roll_link.STL; visual mesh filename=meshes/right_shoulder_roll_link.STL
- link right_shoulder_yaw_link: geometry collision mesh filename=meshes/right_shoulder_yaw_link.STL; visual mesh filename=meshes/right_shoulder_yaw_link.STL
- link right_wrist_pitch_link: geometry collision mesh filename=meshes/right_wrist_pitch_link.STL; visual mesh filename=meshes/right_wrist_pitch_link.STL
- link right_wrist_roll_link: geometry collision mesh filename=meshes/right_wrist_roll_link.STL; visual mesh filename=meshes/right_wrist_roll_link.STL
- link right_wrist_yaw_link: geometry visual mesh filename=meshes/wrist_yaw_link.STL
- link torso_link: geometry collision box size=0.08 0.16 0.1; visual mesh filename=meshes/torso_link.STL
Joints:
- added joint camera_joint: type fixed, parent torso_link, child camera_link, origin xyz=0.11109 0.01750 0.68789 rpy=0 0.8859291283123216 0
- added joint lidar_joint: type fixed, parent torso_link, child lidar_link, origin xyz=0.04874 0 0.67980 rpy=0 0.24015730507441985 0
- joint L_index_intermediate_joint: type fixed -> revolute
- joint L_index_proximal_joint: type fixed -> revolute
- joint L_middle_intermediate_joint: type fixed -> revolute
- joint L_middle_proximal_joint: type fixed -> revolute
- joint L_pinky_intermediate_joint: type fixed -> revolute
- joint L_pinky_proximal_joint: type fixed -> revolute
- joint L_ring_intermediate_joint: type fixed -> revolute
- joint L_ring_proximal_joint: type fixed -> revolute
- joint L_thumb_distal_joint: type fixed -> revolute
- joint L_thumb_intermediate_joint: type fixed -> revolute
- joint L_thumb_proximal_pitch_joint: type fixed -> revolute
- joint L_thumb_proximal_yaw_joint: type fixed -> revolute
- joint R_index_intermediate_joint: type fixed -> revolute
- joint R_index_proximal_joint: type fixed -> revolute
- joint R_middle_intermediate_joint: type fixed -> revolute
- joint R_middle_proximal_joint: type fixed -> revolute
- joint R_pinky_intermediate_joint: type fixed -> revolute
- joint R_pinky_proximal_joint: type fixed -> revolute
- joint R_ring_intermediate_joint: type fixed -> revolute
- joint R_ring_proximal_joint: type fixed -> revolute
- joint R_thumb_distal_joint: type fixed -> revolute
- joint R_thumb_intermediate_joint: type fixed -> revolute
- joint R_thumb_proximal_pitch_joint: type fixed -> revolute
- joint R_thumb_proximal_yaw_joint: type fixed -> revolute
- joint imu_joint: origin xyz=-0.04233868314 0.00166 0.152067 rpy=0 0 0 -> xyz=-0.04452 -0.01891 0.27756 rpy=0 0 0
- joint left_knee_joint: limit lower=-0.26 upper=2.05 effort=300 velocity=14 -> lower=-0.12 upper=2.19 effort=300 velocity=14
- joint left_wrist_pitch_joint: limit lower=-0.47 upper=0.47 effort=19 velocity=31.4 -> lower=-0.4625 upper=0.4625 effort=19 velocity=31.4; origin xyz=0.085 0 0 rpy=0 0 0 -> xyz=0.087 0 0 rpy=0 0 0
- joint right_knee_joint: limit lower=-0.26 upper=2.05 effort=300 velocity=14 -> lower=-0.12 upper=2.19 effort=300 velocity=14
- joint right_wrist_pitch_joint: limit lower=-0.47 upper=0.47 effort=19 velocity=31.4 -> lower=-0.4625 upper=0.4625 effort=19 velocity=31.4; origin xyz=0.085 0 0 rpy=0 0 0 -> xyz=0.087 0 0 rpy=0 0 0
